File: minimal_ltc4296-1/minimal_ltc4296-1.kicad_sch (KiCad schematic)
At the start: 44 parts, among them J1 TBP02R1-381-03BE, J2 TBP02R1-381-03BE, J3 TBP02R1-381-03BE, J4 TBP02R1-381-03BE, J5 TBP02R1-381-03BE, J6 TBP02R1-381-02BE, Q1 100.0 V, Q2 100.0 V, Q3 100.0 V, Q4 100.0 V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

Commit message: Update KiCad PCB file
Parts:
- R12: value 16 mΩ -> 160 mΩ; symbol RESISTORS_PRL1632-_DATA_BASE:R_PRL1632-R016-F-T1 -> RESISTORS_ERJ-B2CF_DATA_BASE:R_ERJ-B2CFR16V; MPN PRL1632-R016-F-T1 -> ERJ-B2CFR16V; Manufacturer Susumu -> Panasonic; Series PRL1632- -> ERJ-B2CF; Symbol Name R_PRL1632-R016-F-T1 -> R_ERJ-B2CFR16V; Trustedparts Search https://www.trustedparts.com/en/search/PRL1632-R016-F-T1 -> https://www.trustedparts.com/en/search/ERJ-B2CFR16V
- R15, R17: value 24 mΩ -> 240 mΩ; symbol RESISTORS_ERJ-B2CF_DATA_BASE:R_ERJ-B2CFR024V -> RESISTORS_ERJ-B2BF_DATA_BASE:R_ERJ-B2BFR24V; MPN ERJ-B2CFR024V -> ERJ-B2BFR24V; Series ERJ-B2CF -> ERJ-B2BF; Symbol Name R_ERJ-B2CFR024V -> R_ERJ-B2BFR24V; Trustedparts Search https://www.trustedparts.com/en/search/ERJ-B2CFR024V -> https://www.trustedparts.com/en/search/ERJ-B2BFR24V
- R16: value 390 mΩ -> 100 mΩ; symbol RESISTORS_ERJ-B2BF_DATA_BASE:R_ERJ-B2BFR39V -> RESISTORS_ERJ-B2CF_DATA_BASE:R_ERJ-B2CFR10V; MPN ERJ-B2BFR39V -> ERJ-B2CFR10V; Series ERJ-B2BF -> ERJ-B2CF; Symbol Name R_ERJ-B2BFR39V -> R_ERJ-B2CFR10V; Trustedparts Search https://www.trustedparts.com/en/search/ERJ-B2BFR39V -> https://www.trustedparts.com/en/search/ERJ-B2CFR10V
- R18: value 24 mΩ -> 1.6 Ω; symbol RESISTORS_ERJ-B2CF_DATA_BASE:R_ERJ-B2CFR024V -> RESISTORS_ERJ-B2BF_DATA_BASE:R_ERJ-B2BF1R6V; MPN ERJ-B2CFR024V -> ERJ-B2BF1R6V; Series ERJ-B2CF -> ERJ-B2BF; Symbol Name R_ERJ-B2CFR024V -> R_ERJ-B2BF1R6V; Trustedparts Search https://www.trustedparts.com/en/search/ERJ-B2CFR024V -> https://www.trustedparts.com/en/search/ERJ-B2BF1R6V
- R19: value 390 mΩ -> 620 mΩ; symbol RESISTORS_ERJ-B2BF_DATA_BASE:R_ERJ-B2BFR39V -> RESISTORS_ERJ-B2BF_DATA_BASE:R_ERJ-B2BFR62V; MPN ERJ-B2BFR39V -> ERJ-B2BFR62V; Symbol Name R_ERJ-B2BFR39V -> R_ERJ-B2BFR62V; Trustedparts Search https://www.trustedparts.com/en/search/ERJ-B2BFR39V -> https://www.trustedparts.com/en/search/ERJ-B2BFR62V
Changed lines of the file:
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@@
 	)
 	(symbol
-		(lib_id "RESISTORS_ERJ-B2CF_DATA_BASE:R_ERJ-B2CFR024V")
+		(lib_id "RESISTORS_ERJ-B2BF_DATA_BASE:R_ERJ-B2BFR24V")
 		(at 287.02 198.12 0)
 		(unit 1)
@@
 			)
 		)
-		(property "Value" "24 mΩ"
+		(property "Value" "240 mΩ"
 			(at 287.02 194.31 0)
 			(effects
@@
 			)
 		)
-		(property "Description" "RES SMD 24 mΩ 1% 0612"
+		(property "Description" "RES SMD 240 mΩ 1% 0612"
 			(at 287.02 208.28 0)
 			(show_name yes)
@@
 			)
 		)
-		(property "MPN" "ERJ-B2CFR024V"
+		(property "MPN" "ERJ-B2BFR24V"
 			(at 287.02 218.44 0)
 			(show_name yes)
@@
 			)
 		)
-		(property "Series" "ERJ-B2CF"
+		(property "Series" "ERJ-B2BF"
 			(at 287.02 223.52 0)
 			(show_name yes)
@@
 			)
 		)
-		(property "Symbol Name" "R_ERJ-B2CFR024V"
+		(property "Symbol Name" "R_ERJ-B2BFR24V"
 			(at 287.02 226.06 0)
 			(show_name yes)
@@
 			)
 		)
-		(property "Trustedparts Search" "https://www.trustedparts.com/en/search/ERJ-B2CFR024V"
+		(property "Trustedparts Search" "https://www.trustedparts.com/en/search/ERJ-B2BFR24V"
 			(at 287.02 233.68 0)
 			(show_name yes)
@@
 	)
 	(symbol
-		(lib_id "RESISTORS_ERJ-B2BF_DATA_BASE:R_ERJ-B2BFR39V")
+		(lib_id "RESISTORS_ERJ-B2CF_DATA_BASE:R_ERJ-B2CFR10V")
 		(at 287.02 157.48 0)
 		(unit 1)
@@
 			)
 		)
-		(property "Value" "390 mΩ"
+		(property "Value" "100 mΩ"
 			(at 287.02 153.67 0)
 			(effects
@@
 			)
 		)
-		(property "Description" "RES SMD 390 mΩ 1% 0612"
+		(property "Description" "RES SMD 100 mΩ 1% 0612"
 			(at 287.02 167.64 0)
 			(show_name yes)
@@
 			)
 		)
-		(property "MPN" "ERJ-B2BFR39V"
+		(property "MPN" "ERJ-B2CFR10V"
 			(at 287.02 177.8 0)
 			(show_name yes)
@@
 			)
 		)
-		(property "Series" "ERJ-B2BF"
+		(property "Series" "ERJ-B2CF"
 			(at 287.02 182.88 0)
 			(show_name yes)
@@
 			)
 		)
-		(property "Symbol Name" "R_ERJ-B2BFR39V"
+		(property "Symbol Name" "R_ERJ-B2CFR10V"
 			(at 287.02 185.42 0)
 			(show_name yes)
@@
 			)
 		)
-		(property "Trustedparts Search" "https://www.trustedparts.com/en/search/ERJ-B2BFR39V"
+		(property "Trustedparts Search" "https://www.trustedparts.com/en/search/ERJ-B2CFR10V"
 			(at 287.02 193.04 0)
 			(show_name yes)
@@
 	)
 	(symbol
-		(lib_id "RESISTORS_ERJ-B2CF_DATA_BASE:R_ERJ-B2CFR024V")
+		(lib_id "RESISTORS_ERJ-B2BF_DATA_BASE:R_ERJ-B2BFR24V")
 		(at 287.02 116.84 0)
 		(unit 1)
@@
 			)
 		)
-		(property "Value" "24 mΩ"
+		(property "Value" "240 mΩ"
 			(at 287.02 113.03 0)
 			(effects
@@
 			)
 		)
-		(property "Description" "RES SMD 24 mΩ 1% 0612"
+		(property "Description" "RES SMD 240 mΩ 1% 0612"
 			(at 287.02 127 0)
 			(show_name yes)
@@
 			)
 		)
-		(property "MPN" "ERJ-B2CFR024V"
+		(property "MPN" "ERJ-B2BFR24V"
 			(at 287.02 137.16 0)
 			(show_name yes)
@@
 			)
 		)
-		(property "Series" "ERJ-B2CF"
+		(property "Series" "ERJ-B2BF"
 			(at 287.02 142.24 0)
 			(show_name yes)
@@
 			)
 		)
-		(property "Symbol Name" "R_ERJ-B2CFR024V"
+		(property "Symbol Name" "R_ERJ-B2BFR24V"
 			(at 287.02 144.78 0)
 			(show_name yes)
@@
 			)
 		)
-		(property "Trustedparts Search" "https://www.trustedparts.com/en/search/ERJ-B2CFR024V"
+		(property "Trustedparts Search" "https://www.trustedparts.com/en/search/ERJ-B2BFR24V"
 			(at 287.02 152.4 0)
 			(show_name yes)
@@
 	)
 	(symbol
-		(lib_id "RESISTORS_ERJ-B2BF_DATA_BASE:R_ERJ-B2BFR39V")
+		(lib_id "RESISTORS_ERJ-B2BF_DATA_BASE:R_ERJ-B2BFR62V")
 		(at 287.02 76.2 0)
 		(unit 1)
@@
 			)
 		)
-		(property "Value" "390 mΩ"
+		(property "Value" "620 mΩ"
 			(at 287.02 72.39 0)
 			(effects
@@
 			)
 		)
-		(property "Description" "RES SMD 390 mΩ 1% 0612"
+		(property "Description" "RES SMD 620 mΩ 1% 0612"
 			(at 287.02 86.36 0)
 			(show_name yes)
@@
 			)
 		)
-		(property "MPN" "ERJ-B2BFR39V"
+		(property "MPN" "ERJ-B2BFR62V"
 			(at 287.02 96.52 0)
 			(show_name yes)
@@
 			)
 		)
-		(property "Symbol Name" "R_ERJ-B2BFR39V"
+		(property "Symbol Name" "R_ERJ-B2BFR62V"
 			(at 287.02 104.14 0)
 			(show_name yes)
@@
 			)
 		)
-		(property "Trustedparts Search" "https://www.trustedparts.com/en/search/ERJ-B2BFR39V"
+		(property "Trustedparts Search" "https://www.trustedparts.com/en/search/ERJ-B2BFR62V"
 			(at 287.02 111.76 0)
 			(show_name yes)
@@
 	)
 	(symbol
-		(lib_id "RESISTORS_PRL1632-_DATA_BASE:R_PRL1632-R016-F-T1")
+		(lib_id "RESISTORS_ERJ-B2CF_DATA_BASE:R_ERJ-B2CFR16V")
 		(at 287.02 99.06 0)
 		(unit 1)
@@
 			)
 		)
-		(property "Value" "16 mΩ"
+		(property "Value" "160 mΩ"
 			(at 287.02 105.41 0)
 			(effects
@@
 			)
 		)
-		(property "Datasheet" "https://www.susumu.co.jp/common/pdf/n_catalog_partition07_en.pdf"
+		(property "Datasheet" "https://industrial.panasonic.com/cdbs/www-data/pdf/RDN0000/AOA0000C325.pdf"
 			(at 287.02 106.68 0)
 			(show_name yes)
@@
 			)
 		)
-		(property "Description" "RES SMD 16 mΩ 1% 0612"
+		(property "Description" "RES SMD 160 mΩ 1% 0612"
 			(at 287.02 109.22 0)
 			(show_name yes)
@@
 			)
 		)
-		(property "MPN" "PRL1632-R016-F-T1"
+		(property "MPN" "ERJ-B2CFR16V"
 			(at 287.02 119.38 0)
 			(show_name yes)
@@
 			)
 		)
-		(property "Manufacturer" "Susumu"
+		(property "Manufacturer" "Panasonic"
 			(at 287.02 121.92 0)
 			(show_name yes)
@@
 			)
 		)
-		(property "Series" "PRL1632-"
+		(property "Series" "ERJ-B2CF"
 			(at 287.02 124.46 0)
 			(show_name yes)
@@
 			)
 		)
-		(property "Symbol Name" "R_PRL1632-R016-F-T1"
+		(property "Symbol Name" "R_ERJ-B2CFR16V"
 			(at 287.02 127 0)
 			(show_name yes)
@@
 			)
 		)
-		(property "Trustedparts Search" "https://www.trustedparts.com/en/search/PRL1632-R016-F-T1"
+		(property "Trustedparts Search" "https://www.trustedparts.com/en/search/ERJ-B2CFR16V"
 			(at 287.02 134.62 0)
 			(show_name yes)
@@
 	)
 	(symbol
-		(lib_id "RESISTORS_ERJ-B2CF_DATA_BASE:R_ERJ-B2CFR024V")
+		(lib_id "RESISTORS_ERJ-B2BF_DATA_BASE:R_ERJ-B2BF1R6V")
 		(at 287.02 35.56 0)
 		(mirror x)
@@
 		(on_board yes)
 		(dnp no)
+		(fields_autoplaced yes)
 		(property "Reference" "R18"
 			(at 287.02 29.21 0)
@@
 			)
 		)
-		(property "Value" "24 mΩ"
+		(property "Value" "1.6 Ω"
 			(at 287.02 31.75 0)
 			(effects
@@
 			)
 		)
-		(property "Description" "RES SMD 24 mΩ 1% 0612"
+		(property "Description" "RES SMD 1.6 Ω 1% 0612"
 			(at 287.02 25.4 0)
 			(show_name yes)
@@
 			)
 		)
-		(property "MPN" "ERJ-B2CFR024V"
+		(property "MPN" "ERJ-B2BF1R6V"
 			(at 287.02 15.24 0)
 			(show_name yes)
@@
 			)
 		)
-		(property "Series" "ERJ-B2CF"
+		(property "Series" "ERJ-B2BF"
 			(at 287.02 10.16 0)
 			(show_name yes)
@@
 			)
 		)
-		(property "Symbol Name" "R_ERJ-B2CFR024V"
+		(property "Symbol Name" "R_ERJ-B2BF1R6V"
 			(at 287.02 7.62 0)
 			(show_name yes)
@@
 			)
 		)
-		(property "Trustedparts Search" "https://www.trustedparts.com/en/search/ERJ-B2CFR024V"
+		(property "Trustedparts Search" "https://www.trustedparts.com/en/search/ERJ-B2BF1R6V"
 			(at 287.02 0 0)
 			(show_name yes)

Commit message: Update KiCad PCB file
Other:
- moved on the sheet: C1, C2, C3, C4, C5, C6, C7, D1, D2, J1, J2, J3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
